Commit message: change to simplebot configuration

File: models/simple_bot.xacro (robot description, xacro)
@@ -1,17 +1,16 @@
 <?xml version="1.0"?>
 <robot name="simple_bot" xmlns:xacro="http://www.ros.org/wiki/xacro">
-  <!-- 기본 파라미터 -->
+  <!-- ===================== 파라미터 ===================== -->
   <xacro:property name="wheel_radius" value="0.033"/>
   <xacro:property name="wheel_width" value="0.025"/>
-  <xacro:property name="body_length" value="0.125"/> <!-- X-axis length: 12.5 cm -->
-  <xacro:property name="body_width"  value="0.115"/> <!-- Y-axis width: 11.5 cm -->
-  <xacro:property name="body_height" value="0.08"/>  <!-- Z-axis height: 8 cm -->
-  <xacro:property name="wheel_base" value="0.08"/> <!-- 앞뒤 바퀴 간격 -->
-  <!-- ===================== base_link ===================== -->
+  <xacro:property name="body_length" value="0.125"/>
+  <xacro:property name="body_width" value="0.115"/>
+  <xacro:property name="body_height" value="0.08"/>
+  <xacro:property name="wheel_base" value="0.08"/>
+  <!-- ===================== Base Link ===================== -->
   <link name="base_link">
     <inertial>
       <mass value="1.0"/>
-      <inertia ixx="0.001" iyy="0.001" izz="0.001"
-              ixy="0.0" ixz="0.0" iyz="0.0"/>
+      <inertia ixx="0.001" iyy="0.001" izz="0.001" ixy="0.0" ixz="0.0" iyz="0.0"/>
     </inertial>
     <visual>
@@ -22,7 +21,12 @@
       <material name="Gray">
         <color rgba="0.6 0.6 0.6 1.0"/>
+        <!-- Gazebo에서 동일하게 보이도록 추가 -->
+        <ambient>0.6 0.6 0.6 1.0</ambient>
+        <diffuse>0.6 0.6 0.6 1.0</diffuse>
+        <specular>0.1 0.1 0.1 1.0</specular>
+        <emissive>0.0 0.0 0.0 1.0</emissive>
       </material>
     </visual>
-    <collision name="base_collision">
+    <collision>
       <geometry>
         <box size="${body_length} ${body_width} ${body_height}"/>
@@ -31,127 +35,40 @@
     </collision>
   </link>
-  <!-- ===================== Left Wheels ===================== -->
-  <!-- Left Front Wheel -->
-  <link name="left_front_wheel_link">
-    <inertial>
-      <mass value="0.2"/>  <!-- 질량 (kg) -->
-      <inertia
-        ixx="0.000056" iyy="0.000056" izz="0.00009"
-        ixy="0.0" ixz="0.0" iyz="0.0"/>
-    </inertial>
-    <visual>
-      <geometry>
-        <cylinder radius="${wheel_radius}" length="${wheel_width}"/>
-      </geometry>
-      <origin xyz="0 0 0" rpy="1.5708 0 0"/>
-      <material name="Black">
-        <color rgba="0 0 0 1"/>
-      </material>
-    </visual>
-    <!-- 💡 물리 충돌 형태 추가 -->
-    <collision name="left_front_wheel_collision">
-      <geometry>
-        <cylinder radius="${wheel_radius}" length="${wheel_width}"/>
-      </geometry>
-      <origin xyz="0 0 0" rpy="1.5708 0 0"/>  <!-- visual과 동일한 회전 적용 -->
-    </collision>
-  </link>
-  <joint name="left_front_wheel_joint" type="continuous">
-    <parent link="base_link"/>
-    <child link="left_front_wheel_link"/>
-    <origin xyz="${wheel_base/2} ${body_width/2 + wheel_width/2} ${wheel_radius}" rpy="0 0 0"/>
-    <axis xyz="0 1 0"/>
-  </joint>
-  <!-- Left Rear Wheel -->
-  <link name="left_rear_wheel_link">
-    <inertial>
-      <mass value="0.2"/>  <!-- 질량 (kg) -->
-      <inertia
-        ixx="0.000056" iyy="0.000056" izz="0.00009"
-        ixy="0.0" ixz="0.0" iyz="0.0"/>
-    </inertial>
-    <visual>
-      <geometry>
-        <cylinder radius="${wheel_radius}" length="${wheel_width}"/>
-      </geometry>
-      <origin xyz="0 0 0" rpy="1.5708 0 0"/>
-      <material name="Black">
-        <color rgba="0 0 0 1"/>
-      </material>
-    </visual>
-    <collision name="left_rear_wheel_collision">
-      <geometry>
-        <cylinder radius="${wheel_radius}" length="${wheel_width}"/>
-      </geometry>
-      <origin xyz="0 0 0" rpy="1.5708 0 0"/>  <!-- visual과 동일한 회전 적용 -->
-    </collision>
-  </link>
-  <joint name="left_rear_wheel_joint" type="continuous">
-    <parent link="base_link"/>
-    <child link="left_rear_wheel_link"/>
-    <origin xyz="-${wheel_base/2} ${body_width/2 + wheel_width/2} ${wheel_radius}" rpy="0 0 0"/>
-    <axis xyz="0 1 0"/>
-  </joint>
-  <!-- ===================== Right Wheels ===================== -->
-  <!-- Right Front Wheel -->
-  <link name="right_front_wheel_link">
-    <inertial>
-      <mass value="0.2"/>  <!-- 질량 (kg) -->
-      <inertia
-        ixx="0.000056" iyy="0.000056" izz="0.00009"
-        ixy="0.0" ixz="0.0" iyz="0.0"/>
-    </inertial>
-    <visual>
-      <geometry>
-        <cylinder radius="${wheel_radius}" length="${wheel_width}"/>
-      </geometry>
-      <origin xyz="0 0 0" rpy="1.5708 0 0"/>
-      <material name="Black">
-        <color rgba="0 0 0 1"/>
-      </material>
-    </visual>
-    <collision name="right_front_wheel_collision">
-      <geometry>
-        <cylinder radius="${wheel_radius}" length="${wheel_width}"/>
-      </geometry>
-      <origin xyz="0 0 0" rpy="1.5708 0 0"/>  <!-- visual과 동일한 회전 적용 -->
-    </collision>
-  </link>
-  <joint name="right_front_wheel_joint" type="continuous">
-    <parent link="base_link"/>
-    <child link="right_front_wheel_link"/>
-    <origin xyz="${wheel_base/2} -${body_width/2 + wheel_width/2} ${wheel_radius}" rpy="0 0 0"/>
-    <axis xyz="0 1 0"/>
-  </joint>
-  <!-- Right Rear Wheel -->
-  <link name="right_rear_wheel_link">
-    <inertial>
-      <mass value="0.2"/>  <!-- 질량 (kg) -->
-      <inertia
-        ixx="0.000056" iyy="0.000056" izz="0.00009"
-        ixy="0.0" ixz="0.0" iyz="0.0"/>
-    </inertial>
-    <visual>
-      <geometry>
-        <cylinder radius="${wheel_radius}" length="${wheel_width}"/>
-      </geometry>
-      <origin xyz="0 0 0" rpy="1.5708 0 0"/>
-      <material name="Black">
-        <color rgba="0 0 0 1"/>
-      </material>
-    <collision name="right_rear_wheel_collision">
-      <geometry>
-        <cylinder radius="${wheel_radius}" length="${wheel_width}"/>
-      </geometry>
-      <origin xyz="0 0 0" rpy="1.5708 0 0"/>  <!-- visual과 동일한 회전 적용 -->
-    </collision>
-    </visual>
-  </link>
-  <joint name="right_rear_wheel_joint" type="continuous">
-    <parent link="base_link"/>
-    <child link="right_rear_wheel_link"/>
-    <origin xyz="-${wheel_base/2} -${body_width/2 + wheel_width/2} ${wheel_radius}" rpy="0 0 0"/>
-    <axis xyz="0 1 0"/>
-  </joint>
+  <!-- ===================== Wheels ===================== -->
+  <xacro:macro name="wheel_link" params="wheel_name x y">
+    <link name="${wheel_name}_link">
+      <inertial>
+        <mass value="0.2"/>
+        <inertia ixx="0.000056" iyy="0.000056" izz="0.00009" ixy="0.0" ixz="0.0" iyz="0.0"/>
+      </inertial>
+      <visual>
+        <geometry>
+          <cylinder radius="${wheel_radius}" length="${wheel_width}"/>
+        </geometry>
+        <origin xyz="0 0 0" rpy="1.5708 0 0"/>
+        <material name="Black">
+          <color rgba="0 0 0 1"/>
+        </material>
+      </visual>
+      <collision>
+        <geometry>
+          <cylinder radius="${wheel_radius}" length="${wheel_width}"/>
+        </geometry>
+        <origin xyz="0 0 0" rpy="1.5708 0 0"/>
+      </collision>
+    </link>
+    <joint name="${wheel_name}_joint" type="continuous">
+      <parent link="base_link"/>
+      <child link="${wheel_name}_link"/>
+      <origin xyz="${x} ${y} ${wheel_radius}" rpy="0 0 0"/>
+      <axis xyz="0 1 0"/>
+    </joint>
+  </xacro:macro>
+  <!-- Left Wheels -->
+  <xacro:wheel_link wheel_name="left_front_wheel" x="${wheel_base/2}" y="${body_width/2 + wheel_width/2}"/>
+  <xacro:wheel_link wheel_name="left_rear_wheel" x="-${wheel_base/2}" y="${body_width/2 + wheel_width/2}"/>
+  <!-- Right Wheels -->
+  <xacro:wheel_link wheel_name="right_front_wheel" x="${wheel_base/2}" y="-${body_width/2 + wheel_width/2}"/>
+  <xacro:wheel_link wheel_name="right_rear_wheel" x="-${wheel_base/2}" y="-${body_width/2 + wheel_width/2}"/>
   <!-- ===================== Ultrasonic Sensor ===================== -->
   <link name="ultrasonic_link">
@@ -160,33 +77,9 @@
         <box size="0.02 0.05 0.02"/>
       </geometry>
-      <origin xyz="0 0 0" rpy="0 0 0"/>  <!-- 자기 중심 -->
       <material name="Yellow">
-        <color rgba="1.0 1.0 0.0 1.0"/>
+        <color rgba="1 1 0 1"/>
       </material>
     </visual>
   </link>
-  <!-- <gazebo reference="ultrasonic_link">
-    <sensor name="ultrasonic_sensor" type="ray">
-      <update_rate>10</update_rate>
-      <ray>
-        <range>
-          <min>0.02</min>
-          <max>2.0</max>
-          <resolution>0.01</resolution>
-        </range>
-        <noise>
-          <type>gaussian</type>
-          <mean>0.0</mean>
-          <stddev>0.01</stddev>
-        </noise>
-      </ray>
-      <plugin name="gazebo_ros_range" filename="libgazebo_ros_range.so">
-        <ros>
-          <namespace>/</namespace>
-          <remapping>~/out:=/ultrasonic/data</remapping>
-        </ros>
-      </plugin>
-    </sensor>
-  </gazebo> -->
   <joint name="ultrasonic_joint" type="fixed">
     <parent link="base_link"/>
@@ -200,38 +93,25 @@
         <box size="0.02 0.05 0.04"/>
       </geometry>
-      <origin xyz="0 0 0" rpy="0 0 0"/>  <!-- 자기 중심 -->
       <material name="Red">
-        <color rgba="1.0 0.0 0.0 1.0"/>
+        <color rgba="1 0 0 1"/>
       </material>
     </visual>
   </link>
-  <!-- <gazebo reference="camera_link">
-    <sensor name="camera_sensor" type="camera">
-      <camera>
-        <horizontal_fov>1.3962634</horizontal_fov>
-        <image>
-          <width>640</width>
-          <height>480</height>
-          <format>R8G8B8</format>
-        </image>
-        <clip>
-          <near>0.05</near>
-          <far>5.0</far>
-        </clip>
-      </camera>
-      <always_on>true</always_on>
-      <update_rate>30</update_rate>
-      <plugin name="gazebo_ros_camera" filename="libgazebo_ros_camera.so">
-        <ros>
-          <namespace>/</namespace>
-          <remapping>~/image_raw:=/camera/image_raw</remapping>
-        </ros>
-      </plugin>
-    </sensor>
-  </gazebo> -->
   <joint name="camera_joint" type="fixed">
     <parent link="base_link"/>
     <child link="camera_link"/>
-    <origin xyz="${(body_length/2) + 0.01} 0 ${body_height*0.7  + 0.02}" rpy="0 0 0"/>
+    <origin xyz="${(body_length/2) + 0.01} 0 ${body_height*0.7 + 0.02}" rpy="0 0 0"/>
   </joint>
+  <!-- ros2_control plugin for Ignition Gazebo -->
+  <gazebo>
+    <!-- Gazebo 플러그인 정의 -->
+    <plugin name="gazebo_ros2_control" filename="libgazebo_ros2_control.so">
+      <ros2_control>
+        <joint name="left_front_wheel_joint"/>
+        <joint name="right_front_wheel_joint"/>
+        <joint name="left_rear_wheel_joint"/>
+        <joint name="right_rear_wheel_joint"/>
+      </ros2_control>
+    </plugin>
+  </gazebo>
 </robot>

File: src/simple_bot/urdf/simple_bot.urdf (robot description, URDF)
Before this commit: robot simple_bot, 7 links, 6 joints
Links:
- link right_rear_wheel_link: geometry visual cylinder length=0.025 radius=0.033
