Commit message: reconfigure in sim

File: models/simple_bot.urdf (robot description, URDF)
Before this commit: robot simple_bot, 7 links, 6 joints
Links:
- link base_link: mass None -> 1.0
- link left_front_wheel_link: mass None -> 0.2; geometry collision cylinder length=0.025 radius=0.033; visual cylinder length=0.025 radius=0.033
- link left_rear_wheel_link: mass None -> 0.2; geometry collision cylinder length=0.025 radius=0.033; visual cylinder length=0.025 radius=0.033
- link right_front_wheel_link: mass None -> 0.2; geometry collision cylinder length=0.025 radius=0.033; visual cylinder length=0.025 radius=0.033
- link right_rear_wheel_link: mass None -> 0.2
Joints:
- removed joint ultrasonic_link
- added joint ultrasonic_joint: type fixed, parent base_link, child ultrasonic_link, origin xyz=0.0725 0 0.04 rpy=0 0 0
- joint camera_joint: origin xyz=0 0 0 rpy=0 0 0 -> xyz=0.0725 0 0.076 rpy=0 0 0

File: models/simple_bot.xacro (robot description, xacro)
@@ -10,17 +10,23 @@
   <!-- ===================== base_link ===================== -->
   <link name="base_link">
+    <inertial>
+      <mass value="1.0"/>
+      <inertia ixx="0.001" iyy="0.001" izz="0.001"
+              ixy="0.0" ixz="0.0" iyz="0.0"/>
+    </inertial>
     <visual>
       <geometry>
         <box size="${body_length} ${body_width} ${body_height}"/>
       </geometry>
-      <origin xyz="0 0 ${body_height/2}" rpy="0 0 0"/>
+      <origin xyz="0 0 ${wheel_radius + body_height/2}" rpy="0 0 0"/>
       <material name="Gray">
         <color rgba="0.6 0.6 0.6 1.0"/>
       </material>
     </visual>
-    <collision>
+    <collision name="base_collision">
       <geometry>
         <box size="${body_length} ${body_width} ${body_height}"/>
       </geometry>
+      <origin xyz="0 0 ${wheel_radius + body_height/2}" rpy="0 0 0"/>
     </collision>
   </link>
@@ -28,13 +34,26 @@
   <!-- Left Front Wheel -->
   <link name="left_front_wheel_link">
-    <visual>
-      <geometry>
-        <cylinder radius="${wheel_radius}" length="${wheel_width}"/>
-      </geometry>
-      <origin xyz="0 0 0" rpy="1.5708 0 0"/>
-      <material name="Black">
-        <color rgba="0 0 0 1"/>
-      </material>
-    </visual>
+    <inertial>
+      <mass value="0.2"/>  <!-- 질량 (kg) -->
+      <inertia
+        ixx="0.000056" iyy="0.000056" izz="0.00009"
+        ixy="0.0" ixz="0.0" iyz="0.0"/>
+    </inertial>
+    <visual>
+      <geometry>
+        <cylinder radius="${wheel_radius}" length="${wheel_width}"/>
+      </geometry>
+      <origin xyz="0 0 0" rpy="1.5708 0 0"/>
+      <material name="Black">
+        <color rgba="0 0 0 1"/>
+      </material>
+    </visual>
+    <!-- 💡 물리 충돌 형태 추가 -->
+    <collision name="left_front_wheel_collision">
+      <geometry>
+        <cylinder radius="${wheel_radius}" length="${wheel_width}"/>
+      </geometry>
+      <origin xyz="0 0 0" rpy="1.5708 0 0"/>  <!-- visual과 동일한 회전 적용 -->
+    </collision>
   </link>
   <joint name="left_front_wheel_joint" type="continuous">
@@ -46,13 +65,25 @@
   <!-- Left Rear Wheel -->
   <link name="left_rear_wheel_link">
-    <visual>
-      <geometry>
-        <cylinder radius="${wheel_radius}" length="${wheel_width}"/>
-      </geometry>
-      <origin xyz="0 0 0" rpy="1.5708 0 0"/>
-      <material name="Black">
-        <color rgba="0 0 0 1"/>
-      </material>
-    </visual>
+    <inertial>
+      <mass value="0.2"/>  <!-- 질량 (kg) -->
+      <inertia
+        ixx="0.000056" iyy="0.000056" izz="0.00009"
+        ixy="0.0" ixz="0.0" iyz="0.0"/>
+    </inertial>
+    <visual>
+      <geometry>
+        <cylinder radius="${wheel_radius}" length="${wheel_width}"/>
+      </geometry>
+      <origin xyz="0 0 0" rpy="1.5708 0 0"/>
+      <material name="Black">
+        <color rgba="0 0 0 1"/>
+      </material>
+    </visual>
+    <collision name="left_rear_wheel_collision">
+      <geometry>
+        <cylinder radius="${wheel_radius}" length="${wheel_width}"/>
+      </geometry>
+      <origin xyz="0 0 0" rpy="1.5708 0 0"/>  <!-- visual과 동일한 회전 적용 -->
+    </collision>
   </link>
   <joint name="left_rear_wheel_joint" type="continuous">
@@ -65,13 +96,25 @@
   <!-- Right Front Wheel -->
   <link name="right_front_wheel_link">
-    <visual>
-      <geometry>
-        <cylinder radius="${wheel_radius}" length="${wheel_width}"/>
-      </geometry>
-      <origin xyz="0 0 0" rpy="1.5708 0 0"/>
-      <material name="Black">
-        <color rgba="0 0 0 1"/>
-      </material>
-    </visual>
+    <inertial>
+      <mass value="0.2"/>  <!-- 질량 (kg) -->
+      <inertia
+        ixx="0.000056" iyy="0.000056" izz="0.00009"
+        ixy="0.0" ixz="0.0" iyz="0.0"/>
+    </inertial>
+    <visual>
+      <geometry>
+        <cylinder radius="${wheel_radius}" length="${wheel_width}"/>
+      </geometry>
+      <origin xyz="0 0 0" rpy="1.5708 0 0"/>
+      <material name="Black">
+        <color rgba="0 0 0 1"/>
+      </material>
+    </visual>
+    <collision name="right_front_wheel_collision">
+      <geometry>
+        <cylinder radius="${wheel_radius}" length="${wheel_width}"/>
+      </geometry>
+      <origin xyz="0 0 0" rpy="1.5708 0 0"/>  <!-- visual과 동일한 회전 적용 -->
+    </collision>
   </link>
   <joint name="right_front_wheel_joint" type="continuous">
@@ -83,12 +126,24 @@
   <!-- Right Rear Wheel -->
   <link name="right_rear_wheel_link">
-    <visual>
-      <geometry>
-        <cylinder radius="${wheel_radius}" length="${wheel_width}"/>
-      </geometry>
-      <origin xyz="0 0 0" rpy="1.5708 0 0"/>
-      <material name="Black">
-        <color rgba="0 0 0 1"/>
-      </material>
+    <inertial>
+      <mass value="0.2"/>  <!-- 질량 (kg) -->
+      <inertia
+        ixx="0.000056" iyy="0.000056" izz="0.00009"
+        ixy="0.0" ixz="0.0" iyz="0.0"/>
+    </inertial>
+    <visual>
+      <geometry>
+        <cylinder radius="${wheel_radius}" length="${wheel_width}"/>
+      </geometry>
+      <origin xyz="0 0 0" rpy="1.5708 0 0"/>
+      <material name="Black">
+        <color rgba="0 0 0 1"/>
+      </material>
+    <collision name="right_rear_wheel_collision">
+      <geometry>
+        <cylinder radius="${wheel_radius}" length="${wheel_width}"/>
+      </geometry>
+      <origin xyz="0 0 0" rpy="1.5708 0 0"/>  <!-- visual과 동일한 회전 적용 -->
+    </collision>
     </visual>
   </link>
@@ -105,5 +160,5 @@
         <box size="0.02 0.05 0.02"/>
       </geometry>
-      <origin xyz="${(body_length/2) + 0.01} 0 ${body_height/4}" rpy="0 0 0"/>
+      <origin xyz="0 0 0" rpy="0 0 0"/>  <!-- 자기 중심 -->
       <material name="Yellow">
         <color rgba="1.0 1.0 0.0 1.0"/>
@@ -111,8 +166,31 @@
     </visual>
   </link>
-  <joint name="ultrasonic_link" type="fixed">
+  <!-- <gazebo reference="ultrasonic_link">
+    <sensor name="ultrasonic_sensor" type="ray">
+      <update_rate>10</update_rate>
+      <ray>
+        <range>
+          <min>0.02</min>
+          <max>2.0</max>
+          <resolution>0.01</resolution>
+        </range>
+        <noise>
+          <type>gaussian</type>
+          <mean>0.0</mean>
+          <stddev>0.01</stddev>
+        </noise>
+      </ray>
+      <plugin name="gazebo_ros_range" filename="libgazebo_ros_range.so">
+        <ros>
+          <namespace>/</namespace>
+          <remapping>~/out:=/ultrasonic/data</remapping>
+        </ros>
+      </plugin>
+    </sensor>
+  </gazebo> -->
+  <joint name="ultrasonic_joint" type="fixed">
     <parent link="base_link"/>
     <child link="ultrasonic_link"/>
-    <origin xyz="0 0 0" rpy="0 0 0"/>
+    <origin xyz="${(body_length/2) + 0.01} 0 ${body_height/4 + 0.02}" rpy="0 0 0"/>
   </joint>
   <!-- ===================== Camera ===================== -->
@@ -122,5 +200,5 @@
         <box size="0.02 0.05 0.04"/>
       </geometry>
-      <origin xyz="${(body_length/2) + 0.01} 0 ${body_height*0.7}" rpy="0 0 0"/>
+      <origin xyz="0 0 0" rpy="0 0 0"/>  <!-- 자기 중심 -->
       <material name="Red">
         <color rgba="1.0 0.0 0.0 1.0"/>
@@ -128,8 +206,32 @@
     </visual>
   </link>
+  <!-- <gazebo reference="camera_link">
+    <sensor name="camera_sensor" type="camera">
+      <camera>
+        <horizontal_fov>1.3962634</horizontal_fov>
+        <image>
+          <width>640</width>
+          <height>480</height>
+          <format>R8G8B8</format>
+        </image>
+        <clip>
+          <near>0.05</near>
+          <far>5.0</far>
+        </clip>
+      </camera>
+      <always_on>true</always_on>
+      <update_rate>30</update_rate>
+      <plugin name="gazebo_ros_camera" filename="libgazebo_ros_camera.so">
+        <ros>
+          <namespace>/</namespace>
+          <remapping>~/image_raw:=/camera/image_raw</remapping>
+        </ros>
+      </plugin>
+    </sensor>
+  </gazebo> -->
   <joint name="camera_joint" type="fixed">
     <parent link="base_link"/>
     <child link="camera_link"/>
-    <origin xyz="0 0 0" rpy="0 0 0"/>
+    <origin xyz="${(body_length/2) + 0.01} 0 ${body_height*0.7  + 0.02}" rpy="0 0 0"/>
   </joint>
 </robot>

Commit message: add gz demo

File: models/simple_bot.urdf (robot description, URDF)
Before this commit: robot simple_bot, 7 links, 6 joints
Links:
- added link odom
Joints:
- added joint odom_to_base: type fixed, parent odom, child base_link, origin xyz=0 0 0 rpy=0 0 0

File: models/simple_bot.xacro (robot description, xacro)
@@ -36,4 +36,13 @@
   </link>
   <!-- ===================== Wheels ===================== -->
+  <!-- odom 프레임 정의 -->
+    <link name="odom"/>
+  <!-- odom → base_link 변환 -->
+  <joint name="odom_to_base" type="fixed">
+    <parent link="odom"/>
+    <child link="base_link"/>
+    <origin xyz="0 0 0" rpy="0 0 0"/>
+  </joint>
+  <!-- ===================== Wheels ===================== -->
   <xacro:macro name="wheel_link" params="wheel_name x y">
     <link name="${wheel_name}_link">
@@ -71,4 +80,47 @@
   <xacro:wheel_link wheel_name="right_front_wheel" x="${wheel_base/2}" y="-${body_width/2 + wheel_width/2}"/>
   <xacro:wheel_link wheel_name="right_rear_wheel" x="-${wheel_base/2}" y="-${body_width/2 + wheel_width/2}"/>
+  <!-- ===================== ros2_control ===================== -->
+  <ros2_control name="GazeboSystem" type="system">
+    <hardware>
+      <plugin>gz_ros2_control/GazeboSystem</plugin>
+    </hardware>
+    <!-- 각 바퀴 joint 정의 -->
+    <joint name="left_front_wheel_joint">
+      <command_interfaces>
+        <interface>velocity</interface>
+      </command_interfaces>
+      <state_interfaces>
+        <interface>position</interface>
+        <interface>velocity</interface>
+      </state_interfaces>
+    </joint>
+    <joint name="left_rear_wheel_joint">
+      <command_interfaces>
+        <interface>velocity</interface>
+      </command_interfaces>
+      <state_interfaces>
+        <interface>position</interface>
+        <interface>velocity</interface>
+      </state_interfaces>
+    </joint>
+    <joint name="right_front_wheel_joint">
+      <command_interfaces>
+        <interface>velocity</interface>
+      </command_interfaces>
+      <state_interfaces>
+        <interface>position</interface>
+        <interface>velocity</interface>
+      </state_interfaces>
+    </joint>
+    <joint name="right_rear_wheel_joint">
+      <command_interfaces>
+        <interface>velocity</interface>
+      </command_interfaces>
+      <state_interfaces>
+        <interface>position</interface>
+        <interface>velocity</interface>
+      </state_interfaces>
+    </joint>
+  </ros2_control>
   <!-- ===================== Ultrasonic Sensor ===================== -->
   <link name="ultrasonic_link">
@@ -103,15 +155,6 @@
     <origin xyz="${(body_length/2) + 0.01} 0 ${body_height*0.7 + 0.02}" rpy="0 0 0"/>
   </joint>
-  <!-- ros2_control plugin for Ignition Gazebo -->
-  <gazebo>
-    <!-- Gazebo 플러그인 정의 -->
-    <plugin name="gazebo_ros2_control" filename="libgazebo_ros2_control.so">
-      <ros2_control>
-        <joint name="left_front_wheel_joint"/>
-        <joint name="right_front_wheel_joint"/>
-        <joint name="left_rear_wheel_joint"/>
-        <joint name="right_rear_wheel_joint"/>
-      </ros2_control>
-    </plugin>
-  </gazebo>
+  <plugin name="gz_ros2_control" filename="libgz_ros2_control-system.so">
+    <parameters>/home/pi/ros2_ws_forpc/config/diff_drive_controller.yaml</parameters>
+  </plugin>
 </robot>
