Commit message: upload good working model ver0.1

File: src/gz_ros2_control/gz_ros2_control_demos/urdf/adeep.urdf (robot description, URDF)
Before this commit: robot adeep_urdf.SLDASM, 7 links, 6 joints
Links:
- link base_link: geometry collision mesh filename=model://adeep/meshes/base_link.STL; visual mesh filename=model://adeep/meshes/base_link.STL
- link camera: geometry collision mesh filename=model://adeep/meshes/camera.STL; visual mesh filename=model://adeep/meshes/camera.STL
- link left_front_wheel: geometry collision mesh filename=model://adeep/meshes/left_front_wheel.STL; visual mesh filename=model://adeep/meshes/left_front_wheel.STL
- link left_rear_wheel: geometry collision mesh filename=model://adeep/meshes/left_rear_wheel.STL; visual mesh filename=model://adeep/meshes/left_rear_wheel.STL
- link right_front_wheel: geometry collision mesh filename=model://adeep/meshes/right_front_wheel.STL; visual mesh filename=model://adeep/meshes/right_front_wheel.STL
- link right_rear_wheel: geometry collision mesh filename=model://adeep/meshes/right_rear_wheel.STL; visual mesh filename=model://adeep/meshes/right_rear_wheel.STL
- link ultrasonic: geometry collision mesh filename=model://adeep/meshes/ultrasonic.STL; visual mesh filename=model://adeep/meshes/ultrasonic.STL
Joints:
- joint camera_joint: origin xyz=0 -0.0725 0.04 rpy=1.5708 0 0 -> xyz=0 -0.0725 0.04 rpy=1.5707963267949 0 0
- joint left_front_wheel_joint: axis 1 0 0 -> -1 0 0
- joint right_front_wheel_joint: axis 1 0 0 -> -1 0 0
- joint right_rear_wheel_joint: axis 1 0 0 -> -1 0 0; origin xyz=-0.0575 0.035 0.015 rpy=2.7498 0 -3.1416 -> xyz=-0.0575 0.035 0.015 rpy=2.74979624140029 0 -3.14159265358979
- joint ultrasonic_joint: origin xyz=0 -0.0725 0.01 rpy=1.5708 0 0 -> xyz=0 -0.0725 0.01 rpy=1.5707963267949 0 0

Commit message: upload unused file

File: src/gz_ros2_control/gz_ros2_control_demos/urdf/adeep.urdf (robot description, URDF)
Before this commit: robot diff_drive, 7 links, 6 joints
Links:
- removed link camera
- removed link ultrasonic
- added link camera_link, mass 0.04; collision mesh filename=model://adeep/meshes/camera.STL; visual mesh filename=model://adeep/meshes/camera.STL
- added link ultrasonic_link, mass 0.02; collision mesh filename=model://adeep/meshes/ultrasonic.STL; visual mesh filename=model://adeep/meshes/ultrasonic.STL
Joints:
- joint camera_joint: child camera -> camera_link
- joint ultrasonic_joint: child ultrasonic -> ultrasonic_link
